File: ATmega32.kicad_pcb (KiCad board)
At the start: 2 copper layers, 23 parts, among them J1 Conn_01x02_Socket, J2 Conn_01x08_Pin, J3 Conn_01x05_Pin, J4 Conn_01x08_Pin, J5 Conn_01x08_Pin, J6 Conn_01x08_Pin, U1 ATmega32A-P, U2 LM7805_TO220, Y1 Crystal

Commit message: edite tracks
Routing:
- net GND: track 48.6 -> 49.3 mm
Changed lines of the file:
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@@
 			(at 7.7216 0.7112 0)
 			(layer "F.SilkS")
+			(hide yes)
 			(effects
 				(font
@@
 	)
 	(segment
-		(start 146.2278 69.7992)
-		(end 134.0104 69.7992)
-		(width 1)
+		(start 130.302 59.69)
+		(end 130.302 66.1416)
+		(width 0.2)
 		(layer "B.Cu")
 		(net 2)
 	)
 	(segment
-		(start 129.794 65.6336)
-		(end 133.985 69.8246)
-		(width 0.2)
+		(start 146.2278 69.7992)
+		(end 134.0104 69.7992)
+		(width 1)
 		(layer "B.Cu")
 		(net 2)
@@
 	)
 	(segment
-		(start 129.794 60.3504)
-		(end 129.794 65.6336)
+		(start 114.4524 46.355)
+		(end 116.967 46.355)
 		(width 0.2)
 		(layer "B.Cu")
@@
 	)
 	(segment
-		(start 115.7986 46.355)
-		(end 129.794 60.3504)
+		(start 130.302 66.1416)
+		(end 133.985 69.8246)
 		(width 0.2)
 		(layer "B.Cu")
@@
 	)
 	(segment
-		(start 114.4524 46.355)
-		(end 115.7986 46.355)
+		(start 116.967 46.355)
+		(end 130.302 59.69)
 		(width 0.2)
 		(layer "B.Cu")

Commit message: Edite design
Parts:
- C1, C2: value 22pF -> 22p; footprint Capacitor_THT:C_Radial_D6.3mm_H11.0mm_P2.50mm -> Capacitor_THT:C_Radial_D4.0mm_H7.0mm_P1.50mm
- C3: footprint Capacitor_THT:C_Radial_D6.3mm_H11.0mm_P2.50mm -> Capacitor_THT:C_Radial_D4.0mm_H7.0mm_P1.50mm
- D1: footprint LED_THT:LED_D3.0mm_FlatTop -> LED_SMD:LED_0805_2012Metric
- Y1: footprint Crystal:Crystal_HC33-U_Vertical -> Crystal:Crystal_C26-LF_D2.1mm_L6.5mm_Vertical
- moved J1 67.5 mm to (160.6, 60.9), turned to 180 degrees
- moved D4 61.5 mm to (160.7, 43.0), turned to 180 degrees
- moved J3 58.8 mm to (103.9, 56.7), turned to 0 degrees
- moved R5 57.6 mm to (155.7, 43.2), turned to 180 degrees
- moved U2 54.5 mm to (156.0, 72.8), turned to 180 degrees
- moved D3 53.9 mm to (160.7, 47.7), turned to 180 degrees
- moved J6 49.0 mm to (107.5, 85.6), turned to 90 degrees
- moved R4 49.0 mm to (155.7, 47.7), turned to 180 degrees
- moved D5 47.0 mm to (108.9, 54.9), turned to 90 degrees
- moved D2 46.7 mm to (160.7, 52.5), turned to 180 degrees
- moved J4 43.6 mm to (121.2, 36.1), turned to -90 degrees
- moved R3 41.4 mm to (155.7, 52.5), turned to 180 degrees
- moved D6 40.0 mm to (108.7, 59.0), turned to -90 degrees
- moved D1 35.3 mm to (155.4, 65.7)
- moved R1 33.8 mm to (152.1, 65.8), turned to 180 degrees
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Connections:
- R3 pad 2: PD2 -> PA7
- R4 pad 2: PD3 -> PA6
- R5 pad 2: PD4 -> PA5
Routing:
- net PD4: track 92.3 -> 12.5 mm
- net PD3: track 81.2 -> 15.5 mm
- net PD2: track 71.5 -> 18.6 mm
- net GND: track 49.3 -> 0.00 mm
- net VCC_MIC: track 84.7 -> 35.6 mm
- net PB0: track 50.9 -> 4.32 mm
- net PD6: track 52.4 -> 6.35 mm
- net PB1: track 48.7 -> 7.17 mm
- net PD5: track 49.3 -> 9.40 mm
- net PB2: track 46.5 -> 10.2 mm
- net DTR: track 78.4 -> 44.2 mm
- net PB3: track 44.3 -> 13.3 mm
- net PB4: track 43.1 -> 16.3 mm
- net PC7: track 4.26 -> 28.8 mm
- net PA7: track 5.28 -> 29.6 mm
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Other:
- board outline added: 63.5 x 58 mm
