File: ATmega32.kicad_sch (KiCad schematic)
At the start: 23 parts, among them J1 Conn_01x02_Socket, J2 Conn_01x08_Pin, J3 Conn_01x05_Pin, J4 Conn_01x08_Pin, J5 Conn_01x08_Pin, J6 Conn_01x08_Pin, U1 ATmega32A-P, U2 LM7805_TO220, Y1 Crystal

Commit message: Edite design
Parts:
- C1, C2, C3: footprint Capacitor_THT:C_Radial_D6.3mm_H11.0mm_P2.50mm -> Capacitor_THT:C_Radial_D4.0mm_H7.0mm_P1.50mm
- D1: footprint LED_THT:LED_D3.0mm_FlatTop -> LED_SMD:LED_0805_2012Metric
- Y1: footprint Crystal:Crystal_HC33-U_Vertical -> Crystal:Crystal_C26-LF_D2.1mm_L6.5mm_Vertical
Connections:
- net PA5: now also R5.2
- net PA6: now also R4.2
- net PA7: now also R3.2
- net PD2: no longer R3.2
- net PD3: no longer R4.2
- net PD4: no longer R5.2
- net VCC_MIC: no longer U1.30 (AVCC)
Changed lines of the file:
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@@
 	(text_box "MIC__ATmega32"
 		(exclude_from_sim no)
-		(at 120.65 13.97 0)
+		(at 120.65 12.7 0)
 		(size 71.12 125.73)
 		(margins 0.9525 0.9525 0.9525 0.9525)
@@
 	(wire
 		(pts
-			(xy 162.56 26.67) (xy 165.1 26.67)
-		)
-		(stroke
-			(width 0)
-			(type default)
-		)
-	)
-	(wire
-		(pts
 			(xy 142.24 63.5) (xy 140.97 63.5)
 		)
@@
 		)
 	)
-	(global_label "PD2"
+	(global_label "PA7"
 		(shape input)
 		(at 95.25 74.93 0)
@@
 		)
 		(property "Intersheetrefs" "${INTERSHEET_REFS}"
-			(at 101.9847 74.93 0)
+			(at 101.8033 74.93 0)
 			(effects
 				(font
@@
 	(global_label "VCC_MIC"
 		(shape input)
-		(at 163.83 26.67 90)
+		(at 162.56 26.67 90)
 		(fields_autoplaced yes)
 		(effects
@@
 		)
 		(property "Intersheetrefs" "${INTERSHEET_REFS}"
-			(at 163.83 15.7624 90)
+			(at 162.56 15.7624 90)
 			(effects
 				(font
@@
 		)
 	)
-	(global_label "PD3"
+	(global_label "PA6"
 		(shape input)
 		(at 95.25 85.09 0)
@@
 		)
 		(property "Intersheetrefs" "${INTERSHEET_REFS}"
-			(at 101.9847 85.09 0)
+			(at 101.8033 85.09 0)
 			(effects
 				(font
@@
 		)
 	)
-	(global_label "PD4"
+	(global_label "PA5"
 		(shape input)
 		(at 95.25 93.98 0)
@@
 		)
 		(property "Intersheetrefs" "${INTERSHEET_REFS}"
-			(at 101.9847 93.98 0)
+			(at 101.8033 93.98 0)
 			(effects
 				(font
@@
 			)
 		)
-		(property "Footprint" "Crystal:Crystal_HC33-U_Vertical"
+		(property "Footprint" "Crystal:Crystal_C26-LF_D2.1mm_L6.5mm_Vertical"
 			(at 137.16 63.5 0)
 			(effects
@@
 			)
 		)
-		(property "Footprint" "Capacitor_THT:C_Radial_D6.3mm_H11.0mm_P2.50mm"
+		(property "Footprint" "Capacitor_THT:C_Radial_D4.0mm_H7.0mm_P1.50mm"
 			(at 143.2052 96.52 0)
 			(effects
@@
 			)
 		)
-		(property "Footprint" "Capacitor_THT:C_Radial_D6.3mm_H11.0mm_P2.50mm"
+		(property "Footprint" "Capacitor_THT:C_Radial_D4.0mm_H7.0mm_P1.50mm"
 			(at 143.2052 72.39 0)
 			(effects
@@
 			)
 		)
-		(property "Footprint" "Capacitor_THT:C_Radial_D6.3mm_H11.0mm_P2.50mm"
+		(property "Footprint" "Capacitor_THT:C_Radial_D4.0mm_H7.0mm_P1.50mm"
 			(at 131.7752 72.39 0)
 			(effects
@@
 			)
 		)
-		(property "Footprint" "LED_THT:LED_D3.0mm_FlatTop"
+		(property "Footprint" "LED_SMD:LED_0805_2012Metric"
 			(at 78.74 115.57 0)
 			(effects
